File: LDO_MON_PMOD_Board_V1/LDO_MON_PMOD_Board_V1.kicad_pcb (KiCad board)
At the start: 2 copper layers, 70.1 x 22 mm, 106 parts, among them J1 3-Pin Harwin, J2 2-Pin Harwin, J3 Conn_01x04, P1 PMOD-Device-x2-Type-Generic-A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, P2 PMOD-Device-x2-Type-Generic-A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, U1 LT3074AV#PBF, U2 LT3074AV#PBF, U3 MAX6373, U4 74LVC1G175, U5 PAC1944x-x4MX, U6 74LVC1G08, U7 AD5272BCP

Commit message: Schematic/PCB Updates.
Parts:
- removed P2: PMOD-Device-x2-Type-Generic-Alt, klib_connectors:pmod_pin_array_6x2
- added C50: 47u, Capacitor_SMD:C_1210_3225Metric, F.Cu at (123.7, 98.8)
- C13, C15, C17, C18, C19, C2, C20, C21, C22, C23, C24, C28, C30, C34, C35, C36, C37, C38, C39, C40, C41, C42, C43, C44, C45, C46, C47, C9, R1, R11, R12, R13, R14, R18, R19, R2, R21, R27, R28, R29, R3, R30, R31, R32, R33, R34, R4, R40, R5: moved to B.Cu
- U4: footprint Package_TO_SOT_SMD:SOT-563 -> Package_TO_SOT_SMD:SOT-23-6
- U6: footprint Package_TO_SOT_SMD:Texas_R-PDSO-G5_DCK-5 -> Package_TO_SOT_SMD:Texas_R-PDSO-N5_DRL-5
- moved R20 70.2 mm to (117.0, 102.2)
- moved R18 70.2 mm to (119.0, 104.2), turned to -90 degrees
- moved R21 66.9 mm to (113.5, 104.2), turned to 180 degrees
- moved U6 64.3 mm to (118.0, 104.2)
- moved C31 63.7 mm to (119.3, 102.2), turned to 180 degrees
- moved R17 62.7 mm to (110.8, 100.8), turned to -90 degrees
- moved J2 62.4 mm to (115.2, 108.2), turned to 90 degrees
- moved C23 61.0 mm to (148.2, 106.0), turned to 180 degrees
- moved C24 60.7 mm to (150.8, 106.0)
- moved R19 59.5 mm to (106.5, 102.7), turned to -90 degrees
- moved R12 59.5 mm to (130.9, 109.8)
- moved R11 59.4 mm to (126.1, 109.8), turned to 180 degrees
- moved C30 57.2 mm to (113.5, 103.2), turned to 180 degrees
- moved C15 56.3 mm to (133.0, 108.5), turned to 90 degrees
- moved C5 55.0 mm to (133.4, 103.0), turned to -135 degrees
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Connections:
- P1 pad 10: unconnected-(P1-P10-Pad10) -> WDI
- P1 pad 3: GPIO -> ALERT_N
- P1 pad 7: unconnected-(P1-P7-Pad7) -> SCL
- P1 pad 8: unconnected-(P1-P8-Pad8) -> SDA
- P1 pad 9: unconnected-(P1-P9-Pad9) -> CNTRL
Routing:
- net BIAS: track 0.00 -> 40.2 mm, vias 0 -> 3
- net GND: track 0.00 -> 25.2 mm, vias 0 -> 19
- net 3V3_PMOD: track 0.00 -> 14.9 mm, vias 0 -> 6
- net SET_RES_NODE: track 0.00 -> 13.5 mm, vias 0 -> 2
- net Net-(U3-~{WDO}): track 0.00 -> 9.17 mm, vias 0 -> 1
- net WDI: track 0.00 -> 8.60 mm, vias 0 -> 2
- net ENABLE: track 0.00 -> 7.83 mm, vias 0 -> 2
- net Net-(JP3-C): track 0.00 -> 5.88 mm
- net Net-(U4-Q): track 0.00 -> 4.55 mm, vias 0 -> 1
- net Net-(JP2-C): track 0.00 -> 4.54 mm
- net Net-(JP1-C): track 0.00 -> 4.45 mm
- net CNTRL: track 0.00 -> 3.60 mm
- net Net-(U2-BIASAF): track 0.00 -> 3.42 mm
- net SCL: track 0.00 -> 2.50 mm, vias 0 -> 2
- net DP_RST_N: track 0.00 -> 2.35 mm
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- added copper zone on In1.Cu, net GND
Other:
- copper layers 2 -> 4

Commit message: PCB Updates.
Parts:
- added C51: 100n, Capacitor_SMD:C_0402_1005Metric, F.Cu at (115.4, 96.9)
- added C52: 100n, Capacitor_SMD:C_0402_1005Metric, F.Cu at (110.8, 97.8)
- added D1: LED, LED_SMD:LED_0402_1005Metric, F.Cu at (105.8, 90.8)
- added D2: LED, LED_SMD:LED_0402_1005Metric, F.Cu at (105.8, 93.1)
- added Q1: MMBT3904, Package_TO_SOT_SMD:SOT-23, B.Cu at (106.2, 98.6)
- added R10: 4k7, Resistor_SMD:R_0402_1005Metric, F.Cu at (108.9, 96.4)
- added R22: 200k, Resistor_SMD:R_0402_1005Metric, F.Cu at (116.4, 95.9)
- added R41: 4k7, Resistor_SMD:R_0402_1005Metric, F.Cu at (108.9, 98.4)
- added R42: 1k, Resistor_SMD:R_0402_1005Metric, F.Cu at (103.6, 90.8)
- added R43: 4k7, Resistor_SMD:R_0402_1005Metric, B.Cu at (107.7, 96.0)
- added R44: 1k, Resistor_SMD:R_0402_1005Metric, B.Cu at (104.4, 96.6)
- added U8: PCA9306, Package_SO:VSSOP-8_2.3x2mm_P0.5mm, F.Cu at (114.4, 98.7)
- moved R7 9.18 mm to (116.3, 100.6)
- moved TP1 5.72 mm to (118.2, 91.0)
- moved TP2 5.72 mm to (118.2, 93.8)
- moved R6 5.45 mm to (117.3, 98.5), turned to -90 degrees
- moved TP3 3.05 mm to (119.9, 99.5)
- moved TP4 3.05 mm to (119.9, 96.8)
- moved R9 2.92 mm to (116.2, 92.3)
- moved C46 2.92 mm to (114.0, 95.0)
- moved C47 2.92 mm to (114.0, 96.0)
- moved C48 2.92 mm to (113.7, 95.5)
- moved C49 2.92 mm to (113.9, 89.9)
- moved R37 2.92 mm to (109.2, 91.4)
- moved R38 2.92 mm to (111.1, 95.0)
- moved U7 2.92 mm to (113.0, 92.4)
- moved R1 1.61 mm to (125.2, 100.5)
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Connections:
- C34 pad 1: Net-(U5-SENSE1+) -> SENSE_1_P_FILT
- C34 pad 2: Net-(U5-SENSE1-) -> SENSE_1_N_FILT
- C35 pad 1: Net-(U5-SENSE1+) -> SENSE_1_P_FILT
- C36 pad 1: Net-(U5-SENSE1-) -> SENSE_1_N_FILT
- C37 pad 1: Net-(U5-SENSE2+) -> SENSE_2_P_FILT
- C37 pad 2: Net-(U5-SENSE2-) -> SENSE_2_N_FILT
- C38 pad 1: Net-(U5-SENSE2+) -> SENSE_2_P_FILT
- C39 pad 1: Net-(U5-SENSE2-) -> SENSE_2_N_FILT
- C40 pad 1: Net-(U5-SENSE3+) -> SENSE_3_P_FILT
- C40 pad 2: Net-(U5-SENSE3-) -> SENSE_3_N_FILT
- C41 pad 1: Net-(U5-SENSE3+) -> SENSE_3_P_FILT
- C42 pad 1: Net-(U5-SENSE3-) -> SENSE_3_N_FILT
- C43 pad 1: Net-(U5-SENSE4+) -> SENSE_4_P_FILT
- C43 pad 2: Net-(U5-SENSE4-) -> SENSE_4_N_FILT
- C44 pad 1: Net-(U5-SENSE4+) -> SENSE_4_P_FILT
- C45 pad 1: Net-(U5-SENSE4-) -> SENSE_4_N_FILT
- P1 pad 4: DP_RST_N -> CNTRL
- P1 pad 7: SCL -> DP_RST_N
- P1 pad 8: SDA -> SCL
- P1 pad 9: CNTRL -> SDA
- R27 pad 1: Net-(U5-SENSE1-) -> SENSE_1_N_FILT
- R28 pad 1: Net-(U5-SENSE1+) -> SENSE_1_P_FILT
- R29 pad 1: Net-(U5-SENSE2+) -> SENSE_2_P_FILT
- R30 pad 1: Net-(U5-SENSE2-) -> SENSE_2_N_FILT
- R31 pad 1: Net-(U5-SENSE3+) -> SENSE_3_P_FILT
- R32 pad 1: Net-(U5-SENSE3-) -> SENSE_3_N_FILT
- R33 pad 1: Net-(U5-SENSE4+) -> SENSE_4_P_FILT
- R34 pad 1: Net-(U5-SENSE4-) -> SENSE_4_N_FILT
- R6 pad 2: SCL -> SCL_HV
- R7 pad 2: SDA -> SDA_HV
- U1 pad 4: SCL -> SCL_HV
- U1 pad 5: SDA -> SDA_HV
- U2 pad 4: SCL -> SCL_HV
- U2 pad 5: SDA -> SDA_HV
- U5 pad 10: Net-(U5-SENSE4+) -> SENSE_1_P_FILT
- U5 pad 11: Net-(U5-SENSE1+) -> SENSE_3_P_FILT
- U5 pad 12: Net-(U5-SENSE1-) -> SENSE_3_N_FILT
- U5 pad 13: Net-(U5-SENSE2+) -> SENSE_4_P_FILT
- U5 pad 14: Net-(U5-SENSE2-) -> SENSE_4_N_FILT
- U5 pad 7: Net-(U5-SENSE3-) -> SENSE_2_N_FILT
- U5 pad 8: Net-(U5-SENSE3+) -> SENSE_2_P_FILT
- U5 pad 9: Net-(U5-SENSE4-) -> SENSE_1_N_FILT
Routing:
- net GND: track 25.2 -> 79.5 mm, vias 19 -> 72
- net ALERT_N: track 1.80 -> 49.7 mm
- net SDA: track 1.80 -> 47.8 mm, vias 2 -> 3
- net SCL: track 2.50 -> 43.9 mm, vias 2 -> 3
- net SLOW: track 0.00 -> 32.7 mm, vias 0 -> 1
- net SCL_HV: track 0.00 -> 32.2 mm, vias 0 -> 3
- net PAC_EN: track 0.00 -> 30.1 mm, vias 0 -> 1
- net SDA_HV: track 0.00 -> 28.2 mm, vias 0 -> 3
- net BIAS: track 40.2 -> 68.0 mm, vias 3 -> 5
- net SENSE_3_N_FILT: track 0.00 -> 27.5 mm, vias 0 -> 1
- net SENSE_4_P_FILT: track 0.00 -> 27.1 mm, vias 0 -> 1
- net ENABLE: track 7.83 -> 34.9 mm, vias 2 -> 1
- net SENSE_4_N_FILT: track 0.00 -> 27.0 mm, vias 0 -> 1
- net SENSE_3_P_FILT: track 0.00 -> 26.4 mm, vias 0 -> 1
- net SENSE_2_N_FILT: track 0.00 -> 23.6 mm, vias 0 -> 1
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- added copper zone on F.Cu, net 3V3_PMOD
- added copper zone on In2.Cu, net 3V3_PMOD
- added copper zone on B.Cu, net GND
- added copper zone on F.Cu, net GND
- added copper zone on In4.Cu, net GND
- added copper zone on F.Cu, net OUT_1
- added copper zone on F.Cu, net OUT_2
- added copper zone on B.Cu, net SENSE_1_N
- added copper zone on F.Cu, net SENSE_1_N
- added copper zone on F.Cu, net SENSE_3_N
- added copper zone on F.Cu, net SENSE_4_N
- added copper zone on In3.Cu, net SENSE_4_N
- added copper zone on F.Cu, net SENSE_4_P
Other:
- copper layers 4 -> 6
