File: LDO_MON_PMOD_Board_V1/LDO_MON_PMOD_Board_V1.kicad_pcb (KiCad board)
At the start: 6 copper layers, 70.1 x 22 mm, 118 parts, among them J1 3-Pin Harwin, J2 2-Pin Harwin, J3 Conn_01x04, P1 PMOD-Device-x2-Type-Generic-A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, Q1 MMBT3904, U1 LT3074AV#PBF, U2 LT3074AV#PBF, U3 MAX6373, U4 74LVC1G175, U5 PAC1944x-x4MX, U6 74LVC1G08, U7 AD5272BCP, U8 PCA9306

Commit message: Fixed problem with watchdog enable bypass. Updated schematic/PCB/gerbers. No change to placement or BOM.
Connections:
- J2 pad 1: 3V3_PMOD -> ENABLE
- J2 pad 2: ENABLE -> Net-(J2-Pin_2)
- U6 pad 4: ENABLE -> Net-(J2-Pin_2)
Routing:
- net ENABLE: track 34.9 -> 39.5 mm
- net Net-(J2-Pin_2): track 0.00 -> 3.90 mm
Changed lines of the file:
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@@
 		(sheetname "/")
 		(sheetfile "LDO_MON_PMOD_Board_V1.kicad_sch")
+		(units
+			(unit
+				(name "A")
+				(pins "1" "2" "3")
+			)
+		)
 		(zone_connect 1)
 		(attr exclude_from_bom allow_soldermask_bridges)
@@
 		(sheetname "/")
 		(sheetfile "LDO_MON_PMOD_Board_V1.kicad_sch")
+		(units
+			(unit
+				(name "A")
+				(pins "11" "12" "13" "14" "8" "7" "10" "9" "2" "3" "17" "4" "5" "16"
+					"1" "15" "6"
+				)
+			)
+		)
 		(attr smd)
 		(duplicate_pad_numbers_are_jumpers no)
@@
 			(layers "F.Cu" "F.Mask" "F.Paste")
 			(roundrect_rratio 0.1666666667)
-			(net "ENABLE")
+			(net "Net-(J2-Pin_2)")
 			(pintype "output")
 		)
@@
 		(sheetname "/")
 		(sheetfile "LDO_MON_PMOD_Board_V1.kicad_sch")
+		(units
+			(unit
+				(name "A")
+				(pins "1" "2" "3")
+			)
+		)
 		(zone_connect 1)
 		(attr exclude_from_bom allow_soldermask_bridges)
@@
 		(sheetname "/")
 		(sheetfile "LDO_MON_PMOD_Board_V1.kicad_sch")
+		(units
+			(unit
+				(name "A")
+				(pins "1" "2" "3" "4")
+			)
+		)
 		(attr through_hole)
 		(duplicate_pad_numbers_are_jumpers no)
@@
 			(layers "*.Cu" "*.Mask")
 			(remove_unused_layers no)
-			(net "3V3_PMOD")
+			(net "ENABLE")
 			(pinfunction "Pin_1_1")
 			(pintype "passive")
@@
 			(layers "*.Cu" "*.Mask")
 			(remove_unused_layers no)
-			(net "ENABLE")
+			(net "Net-(J2-Pin_2)")
 			(pinfunction "Pin_2_2")
 			(pintype "passive")
@@
 		(sheetname "/")
 		(sheetfile "LDO_MON_PMOD_Board_V1.kicad_sch")
+		(units
+			(unit
+				(name "A")
+				(pins "1" "2" "3")
+			)
+		)
 		(zone_connect 1)
 		(attr exclude_from_bom allow_soldermask_bridges)
@@
 	)
 	(segment
+		(start 119 109.7)
+		(end 116.725 109.7)
+		(width 0.1)
+		(layer "F.Cu")
+		(net "ENABLE")
+	)
+	(segment
 		(start 122.4 102.3)
 		(end 120 104.7)
@@
 	)
 	(segment
-		(start 126.6 99.5)
-		(end 126.6 100.15)
+		(start 116.725 109.7)
+		(end 115.225 108.2)
 		(width 0.1)
 		(layer "F.Cu")
@@
 	)
 	(segment
-		(start 117.765 108.2)
-		(end 118.74 107.225)
-		(width 0.2)
+		(start 126.6 99.5)
+		(end 126.6 100.15)
+		(width 0.1)
 		(layer "F.Cu")
 		(net "ENABLE")
@@
 	)
 	(segment
-		(start 118.74 104.7)
-		(end 120 104.7)
-		(width 0.2)
+		(start 126.6 100.15)
+		(end 126.6 101.6)
+		(width 0.1)
 		(layer "F.Cu")
 		(net "ENABLE")
 	)
 	(segment
-		(start 118.74 107.225)
-		(end 118.74 104.7)
-		(width 0.2)
+		(start 120 104.7)
+		(end 120 108.7)
+		(width 0.1)
 		(layer "F.Cu")
 		(net "ENABLE")
 	)
 	(segment
-		(start 126.6 100.15)
-		(end 126.6 101.6)
+		(start 120 108.7)
+		(end 119 109.7)
 		(width 0.1)
 		(layer "F.Cu")
@@
 		(net "Net-(Q1-C)")
 	)
+	(segment
+		(start 118.74 104.7)
+		(end 118.74 107.225)
+		(width 0.15)
+		(layer "F.Cu")
+		(net "Net-(J2-Pin_2)")
+	)
+	(segment
+		(start 118.74 107.225)
+		(end 117.765 108.2)
+		(width 0.15)
+		(layer "F.Cu")
+		(net "Net-(J2-Pin_2)")
+	)
 	(zone

Commit message: Fixed/removed alert_n flag at wrong voltage potential.
Connections:
- P1 pad 3: ALERT_N -> unconnected-(P1-P3-Pad3)
Routing:
- net ALERT_N: track 49.7 -> 14.8 mm
Changed lines of the file:
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@@
 			(layers "*.Cu" "*.Mask")
 			(remove_unused_layers no)
-			(net "ALERT_N")
+			(net "unconnected-(P1-P3-Pad3)")
 			(pinfunction "P3_3")
-			(pintype "passive")
+			(pintype "passive+no_connect")
 		)
 		(pad "4" thru_hole circle
@@
 	)
 	(segment
-		(start 124.4 102.4)
-		(end 115.8 93.8)
-		(width 0.1)
-		(layer "B.Cu")
-		(net "ALERT_N")
-	)
-	(segment
-		(start 103.9 92.6)
-		(end 103.3 93.2)
-		(width 0.1)
-		(layer "B.Cu")
-		(net "ALERT_N")
-	)
-	(segment
 		(start 129.35 108.7)
 		(end 129.7 108.7)
@@
 	)
 	(segment
-		(start 126.61 102.4)
-		(end 124.4 102.4)
-		(width 0.1)
-		(layer "B.Cu")
-		(net "ALERT_N")
-	)
-	(segment
 		(start 128.25 101.35)
 		(end 127.85 101.75)
@@
 	)
 	(segment
-		(start 115.8 93.8)
-		(end 106.8 93.8)
-		(width 0.1)
-		(layer "B.Cu")
-		(net "ALERT_N")
-	)
-	(segment
 		(start 129.7 108.7)
 		(end 130.2 108.2)
@@
 	)
 	(segment
-		(start 103.3 93.2)
-		(end 103.3 96.7)
-		(width 0.1)
-		(layer "B.Cu")
-		(net "ALERT_N")
-	)
-	(segment
-		(start 103.3 96.7)
-		(end 101.27 98.73)
-		(width 0.1)
-		(layer "B.Cu")
-		(net "ALERT_N")
-	)
-	(segment
-		(start 105.6 92.6)
-		(end 103.9 92.6)
-		(width 0.1)
-		(layer "B.Cu")
-		(net "ALERT_N")
-	)
-	(segment
-		(start 127.26 101.75)
-		(end 126.61 102.4)
-		(width 0.1)
-		(layer "B.Cu")
-		(net "ALERT_N")
-	)
-	(segment
 		(start 128.25 100.8)
 		(end 128.25 101.35)
@@
 	)
 	(segment
-		(start 106.8 93.8)
-		(end 105.6 92.6)
-		(width 0.1)
-		(layer "B.Cu")
-		(net "ALERT_N")
-	)
-	(segment
 		(start 117.9 103.35)
 		(end 117.6 103.05)
@@
 	)
 	(segment
-		(start 119 109.7)
-		(end 116.725 109.7)
-		(width 0.1)
-		(layer "F.Cu")
-		(net "ENABLE")
-	)
-	(segment
-		(start 122.4 102.3)
-		(end 120 104.7)
-		(width 0.1)
-		(layer "F.Cu")
-		(net "ENABLE")
-	)
-	(segment
-		(start 125.9 102.3)
-		(end 122.4 102.3)
-		(width 0.1)
-		(layer "F.Cu")
-		(net "ENABLE")
-	)
-	(segment
-		(start 116.725 109.7)
-		(end 115.225 108.2)
-		(width 0.1)
-		(layer "F.Cu")
-		(net "ENABLE")
-	)
-	(segment
-		(start 126.6 99.5)
-		(end 126.6 100.15)
-		(width 0.1)
-		(layer "F.Cu")
-		(net "ENABLE")
-	)
-	(segment
-		(start 126.6 101.6)
-		(end 125.9 102.3)
-		(width 0.1)
-		(layer "F.Cu")
-		(net "ENABLE")
-	)
-	(segment
-		(start 126.6 100.15)
-		(end 126.6 101.6)
-		(width 0.1)
-		(layer "F.Cu")
-		(net "ENABLE")
-	)
-	(segment
-		(start 120 104.7)
-		(end 120 108.7)
-		(width 0.1)
+		(start 118.74 104.7)
+		(end 118.74 107.225)
+		(width 0.15)
 		(layer "F.Cu")
-		(net "ENABLE")
+		(net "Net-(J2-Pin_2)")
 	)
 	(segment
-		(start 120 108.7)
-		(end 119 109.7)
-		(width 0.1)
+		(start 118.74 107.225)
+		(end 117.765 108.2)
+		(width 0.15)
 		(layer "F.Cu")
-		(net "ENABLE")
-	)
-	(via
-		(at 120 104.7)
-		(size 0.5)
-		(drill 0.25)
-		(layers "F.Cu" "B.Cu")
-		(net "ENABLE")
-	)
-	(segment
-		(start 118.9 99.7)
-		(end 118.9 102.4)
-		(width 0.1)
-		(layer "B.Cu")
-		(net "ENABLE")
-	)
-	(segment
-		(start 118.9 102.4)
-		(end 118.4 102.9)
-		(width 0.1)
-		(layer "B.Cu")
-		(net "ENABLE")
-	)
-	(segment
-		(start 118.5 99.3)
-		(end 118.9 99.7)
-		(width 0.1)
-		(layer "B.Cu")
-		(net "ENABLE")
-	)
-	(segment
-		(start 119.01 104.7)
-		(end 119 104.71)
-		(width 0.2)
-		(layer "B.Cu")
-		(net "ENABLE")
-	)
-	(segment
-		(start 120.94 104.7)
-		(end 120.99 104.75)
-		(width 0.2)
-		(layer "B.Cu")
-		(net "ENABLE")
-	)
-	(segment
-		(start 118.4 102.9)
-		(end 118.4 104.11)
-		(width 0.1)
-		(layer "B.Cu")
-		(net "ENABLE")
-	)
-	(segment
-		(start 108.21 96)
-		(end 111.8 96)
-		(width 0.1)
-		(layer "B.Cu")
-		(net "ENABLE")
-	)
-	(segment
-		(start 118 99.3)
-		(end 118.5 99.3)
-		(width 0.1)
-		(layer "B.Cu")
-		(net "ENABLE")
-	)
-	(segment
-		(start 120 104.7)
-		(end 119.01 104.7)
-		(width 0.2)
-		(layer "B.Cu")
-		(net "ENABLE")
-	)
-	(segment
-		(start 111.8 96)
-		(end 113.9 98.1)
-		(width 0.1)
-		(layer "B.Cu")
-		(net "ENABLE")
-	)
-	(segment
-		(start 116.8 98.1)
-		(end 118 99.3)
-		(width 0.1)
-		(layer "B.Cu")
-		(net "ENABLE")
-	)
-	(segment
-		(start 120 104.7)
-		(end 120.94 104.7)
-		(width 0.2)
-		(layer "B.Cu")
-		(net "ENABLE")
-	)
-	(segment
-		(start 118.4 104.11)
-		(end 119 104.71)
-		(width 0.1)
-		(layer "B.Cu")
-		(net "ENABLE")
-	)
-	(segment
-		(start 113.9 98.1)
-		(end 116.8 98.1)
-		(width 0.1)
-		(layer "B.Cu")
-		(net "ENABLE")
+		(net "Net-(J2-Pin_2)")
 	)
 	(segment
@@
 	)
 	(segment
+		(start 119 109.7)
+		(end 116.725 109.7)
+		(width 0.1)
+		(layer "F.Cu")
+		(net "ENABLE")
+	)
+	(segment
+		(start 122.4 102.3)
+		(end 120 104.7)
+		(width 0.1)
+		(layer "F.Cu")
+		(net "ENABLE")
+	)
+	(segment
+		(start 125.9 102.3)
+		(end 122.4 102.3)
+		(width 0.1)
+		(layer "F.Cu")
+		(net "ENABLE")
+	)
+	(segment
+		(start 116.725 109.7)
+		(end 115.225 108.2)
+		(width 0.1)
+		(layer "F.Cu")
+		(net "ENABLE")
+	)
+	(segment
+		(start 126.6 99.5)
+		(end 126.6 100.15)
+		(width 0.1)
+		(layer "F.Cu")
+		(net "ENABLE")
+	)
+	(segment
+		(start 126.6 101.6)
+		(end 125.9 102.3)
+		(width 0.1)
+		(layer "F.Cu")
+		(net "ENABLE")
+	)
+	(segment
+		(start 126.6 100.15)
+		(end 126.6 101.6)
+		(width 0.1)
+		(layer "F.Cu")
+		(net "ENABLE")
+	)
+	(segment
+		(start 120 104.7)
+		(end 120 108.7)
+		(width 0.1)
+		(layer "F.Cu")
+		(net "ENABLE")
+	)
+	(segment
+		(start 120 108.7)
+		(end 119 109.7)
+		(width 0.1)
+		(layer "F.Cu")
+		(net "ENABLE")
+	)
+	(via
+		(at 120 104.7)
+		(size 0.5)
+		(drill 0.25)
+		(layers "F.Cu" "B.Cu")
+		(net "ENABLE")
+	)
+	(segment
+		(start 118.9 99.7)
+		(end 118.9 102.4)
+		(width 0.1)
+		(layer "B.Cu")
+		(net "ENABLE")
+	)
+	(segment
+		(start 118.9 102.4)
+		(end 118.4 102.9)
+		(width 0.1)
+		(layer "B.Cu")
+		(net "ENABLE")
+	)
+	(segment
+		(start 118.5 99.3)
+		(end 118.9 99.7)
+		(width 0.1)
+		(layer "B.Cu")
+		(net "ENABLE")
+	)
+	(segment
+		(start 119.01 104.7)
+		(end 119 104.71)
+		(width 0.2)
+		(layer "B.Cu")
+		(net "ENABLE")
+	)
+	(segment
+		(start 120.94 104.7)
+		(end 120.99 104.75)
+		(width 0.2)
+		(layer "B.Cu")
+		(net "ENABLE")
+	)
+	(segment
+		(start 118.4 102.9)
+		(end 118.4 104.11)
+		(width 0.1)
+		(layer "B.Cu")
+		(net "ENABLE")
+	)
+	(segment
+		(start 108.21 96)
+		(end 111.8 96)
+		(width 0.1)
+		(layer "B.Cu")
+		(net "ENABLE")
+	)
+	(segment
+		(start 118 99.3)
+		(end 118.5 99.3)
+		(width 0.1)
+		(layer "B.Cu")
+		(net "ENABLE")
+	)
+	(segment
+		(start 120 104.7)
+		(end 119.01 104.7)
+		(width 0.2)
+		(layer "B.Cu")
+		(net "ENABLE")
+	)
+	(segment
+		(start 111.8 96)
+		(end 113.9 98.1)
+		(width 0.1)
+		(layer "B.Cu")
+		(net "ENABLE")
+	)
+	(segment
+		(start 116.8 98.1)
+		(end 118 99.3)
+		(width 0.1)
+		(layer "B.Cu")
+		(net "ENABLE")
+	)
+	(segment
+		(start 120 104.7)
+		(end 120.94 104.7)
+		(width 0.2)
+		(layer "B.Cu")
+		(net "ENABLE")
+	)
+	(segment
+		(start 118.4 104.11)
+		(end 119 104.71)
+		(width 0.1)
+		(layer "B.Cu")
+		(net "ENABLE")
+	)
+	(segment
+		(start 113.9 98.1)
+		(end 116.8 98.1)
+		(width 0.1)
+		(layer "B.Cu")
+		(net "ENABLE")
+	)
+	(segment
 		(start 104.12 90.81)
 		(end 104.11 90.8)
@@
 		(net "Net-(Q1-C)")
 	)
-	(segment
-		(start 118.74 104.7)
-		(end 118.74 107.225)
-		(width 0.15)
-		(layer "F.Cu")
-		(net "Net-(J2-Pin_2)")
-	)
-	(segment
-		(start 118.74 107.225)
-		(end 117.765 108.2)
-		(width 0.15)
-		(layer "F.Cu")
-		(net "Net-(J2-Pin_2)")
-	)
 	(zone
